Commit message: changes on jackal simulator (likely from Jackal itself).

File: jackal_description/urdf/accessories/bridge_plate.urdf.xacro (robot description, xacro)
@@ -1,11 +1,17 @@
 <?xml version="1.0"?>
-<robot xmlns:xacro="http://ros.org/wiki/xacro">
-  <xacro:macro name="bridge_plate" params="mount height">
-    <joint name="${mount}_mount_to_${mount}_bridge" type="fixed">
-      <parent link="${mount}_mount"/>
-      <child link="${mount}_bridge"/>
+<robot xmlns:xacro="http://www.ros.org/wiki/xacro">
+  <xacro:macro name="bridge_plate" params="prefix parent height *origin">
+    <link name="${prefix}_bridge_base"/>
+    <joint name="${prefix}_bridge_base_joint" type="fixed">
+      <parent link="${parent}"/>
+      <child link="${prefix}_bridge_base" />
+      <xacro:insert_block name="origin" />
+    </joint>
+    <joint name="${prefix}_bridge_joint" type="fixed">
+      <parent link="${prefix}_bridge_base"/>
+      <child link="${prefix}_bridge"/>
       <origin xyz="0.0 0.0 ${height}" rpy="0 0 0"/>
     </joint>
-    <link name="${mount}_bridge">
+    <link name="${prefix}_bridge">
       <visual>
         <origin xyz="0 0 0" rpy="1.5707 0.0 1.5707" />
@@ -16,5 +22,5 @@
       </visual>
     </link>
-    <standoff_box mount="${mount}" height="${height}" />
+    <xacro:standoff_box prefix="${prefix}" parent="${prefix}_bridge_base" height="${height}" />
   </xacro:macro>
 </robot>

File: jackal_description/urdf/accessories/sick_lms1xx_inverted_mount.urdf.xacro (robot description, xacro)
@@ -25,8 +25,13 @@
 SOFTWARE, EVEN IF ADVISED OF THE POSSIBILITY OF SUCH DAMAGE.
 -->
-<robot xmlns:xacro="http://ros.org/wiki/xacro">
+<robot xmlns:xacro="http://www.ros.org/wiki/xacro">
   <xacro:include filename="$(find lms1xx)/urdf/sick_lms1xx.urdf.xacro" />
-  <xacro:macro name="sick_lms1xx_mount" params="prefix topic">
-    <sick_lms1xx frame="${prefix}_laser" topic="${topic}" />
+  <xacro:macro name="sick_lms1xx_inverted_mount" params="prefix topic parent_link *origin">
+    <xacro:sick_lms1xx frame="${prefix}_laser" topic="${topic}" />
+    <joint name="${prefix}_laser_mount_joint" type="fixed">
+      <xacro:insert_block name="origin" />
+      <parent link="${parent_link}" />
+      <child link="${prefix}_laser_mount" />
+    </joint>
     <link name="${prefix}_laser_mount">
       <visual>
@@ -34,5 +39,5 @@
         <geometry>
           <!-- Origin of this mesh is the base of the bracket. -->
-          <mesh filename="package://jackal_description/meshes/sick-lms1xx-bracket.stl" />
+          <mesh filename="package://jackal_description/meshes/sick-lms1xx-inverted-bracket.stl" />
         </geometry>
         <material name="dark_grey" />
@@ -41,5 +46,5 @@
     <joint name="${prefix}_laser_joint" type="fixed">
       <!-- This offset is from the base of the bracket to the LIDAR's focal point. -->
-      <origin xyz="0 0 0.149" rpy="0 0 0" />
+      <origin xyz="0.04 0 0.066" rpy="3.141592 0 0" />
       <parent link="${prefix}_laser_mount" />
       <child link="${prefix}_laser" />

File: jackal_description/urdf/jackal.urdf.xacro (robot description, xacro)
@@ -43,4 +43,10 @@
     <gazebo reference="${prefix}_wheel_link">
       <material>Gazebo/DarkGrey</material>
+      <selfCollide>false</selfCollide>
+      <mu1 value="0.5"/>
+      <mu2 value="0.5"/>
+      <kp value="10000000.0" />
+      <kd value="1" />
+      <fdir1 value="1 0 0"/>
     </gazebo>
     <joint name="${prefix}_wheel" type="continuous">
@@ -55,5 +61,5 @@
       <type>transmission_interface/SimpleTransmission</type>
       <joint name="${prefix}_wheel">
-        <hardwareInterface>VelocityJointInterface</hardwareInterface>
+        <hardwareInterface>hardware_interface/VelocityJointInterface</hardwareInterface>
       </joint>
       <actuator name="${prefix}_actuator">
@@ -105,21 +111,67 @@
       </inertial>
   </link>
-  <link name="fenders_link">
-    <visual>
-      <origin xyz="0 0 ${footprint_vertical_offset}" rpy="${PI/2} 0 ${PI/2}"/>
-      <geometry>
-        <mesh filename="package://jackal_description/meshes/jackal-fenders.stl"/>
-      </geometry>
-      <material name="yellow" />
-    </visual>
-  </link>
-  <joint name="fenders_joint" type="fixed">
-    <parent link="chassis_link" />
-    <child link="fenders_link" />
-  </joint>
-  <!-- TODO: Make this internal_imu_link or something, and use a mixed-in xacro
-       to supply the joint between it and imu_link. This is important so that imu_link
-       always points to the "active" IMU. When an upgrade IMU is connected, the
-       internal_imu_link should remain, but imu_link should point to the upgrade one. -->
+  <xacro:unless value="$(optenv JACKAL_FRONT_ACCESSORY_FENDER 0)">
+    <link name="front_fender_link">
+      <visual>
+        <geometry>
+          <mesh filename="package://jackal_description/meshes/jackal-fender.stl"/>
+        </geometry>
+        <material name="yellow" />
+      </visual>
+    </link>
+  </xacro:unless>
+  <xacro:if value="$(optenv JACKAL_FRONT_ACCESSORY_FENDER 0)">
+    <link name="front_fender_link">
+      <visual>
+        <geometry>
+          <mesh filename="package://jackal_description/meshes/accessory_fender.stl"/>
+        </geometry>
+        <material name="yellow" />
+      </visual>
+    </link>
+    <link name="front_fender_accessory_link"/>
+    <joint name="front_fender_accessory_joint" type="fixed">
+      <origin xyz="0.25629 0 0.07455" rpy="${PI} 0 0" />
+      <parent link="front_fender_link" />
+      <child link="front_fender_accessory_link" />
+    </joint>
+  </xacro:if>
+  <joint name="front_fender_joint" type="fixed">
+    <origin xyz="0 0 0" rpy="0 0 0"/>
+    <parent link="chassis_link" />
+    <child link="front_fender_link" />
+  </joint>
+  <xacro:unless value="$(optenv JACKAL_REAR_ACCESSORY_FENDER 0)">
+    <link name="rear_fender_link">
+      <visual>
+        <geometry>
+          <mesh filename="package://jackal_description/meshes/jackal-fender.stl"/>
+        </geometry>
+        <material name="yellow" />
+      </visual>
+    </link>
+  </xacro:unless>
+  <xacro:if value="$(optenv JACKAL_REAR_ACCESSORY_FENDER 0)">
+    <link name="rear_fender_link">
+      <visual>
+        <geometry>
+          <mesh filename="package://jackal_description/meshes/accessory_fender.stl"/>
+        </geometry>
+        <material name="yellow" />
+      </visual>
+    </link>
+    <link name="rear_fender_accessory_link"/>
+    <joint name="rear_fender_accessory_joint" type="fixed">
+      <origin xyz="0.25629 0 0.07455" rpy="${PI} 0 0" />
+      <parent link="rear_fender_link" />
+      <child link="rear_fender_accessory_link" />
+    </joint>
+  </xacro:if>
+  <joint name="rear_fender_joint" type="fixed">
+    <origin xyz="0 0 0" rpy="0 0 ${PI}"/>
+    <parent link="chassis_link" />
+    <child link="rear_fender_link" />
+  </joint>
+  <!-- Default Internal IMU Link -->
   <link name="imu_link">
     <inertial>
@@ -133,5 +185,5 @@
     <child link="imu_link" />
   </joint>
-  <!-- TODO: Same note as applies to imu_link -->
+  <!-- Default NAVSAT Link -->
   <link name="navsat_link">
     <visual>
@@ -172,5 +224,15 @@
        default each one to off.-->
   <xacro:include filename="$(find jackal_description)/urdf/accessories.urdf.xacro" />
+  <!-- OutdoorNav -->
+  <xacro:arg name="outdoornav_enabled"       default="$(optenv OUTDOORNAV_ENABLED 0)" />
+  <xacro:arg name="outdoornav_configuration" default="$(optenv OUTDOORNAV_CONFIGURATION standard)" />
+  <!-- OutdoorNav URDF Config -->
+  <xacro:if value="$(arg outdoornav_enabled)">
+    <xacro:include filename="$(find cpr_onav_description)/urdf/outdoornav_description.urdf.xacro" />
+    <xacro:outdoornav_sensors outdoornav_configuration="$(arg outdoornav_configuration)" />
+  </xacro:if>
   <!-- Optional custom includes. -->
   <xacro:include filename="$(optenv JACKAL_URDF_EXTRAS empty.urdf)" />
+  <!-- Optional for Clearpath internal softwares -->
+  <xacro:include filename="$(optenv CPR_URDF_EXTRAS empty.urdf)" />
 </robot>
